Commit message: add mocap link for vicon tracking

File: jackal_description/urdf/sensors_pic4ser.urdf (robot description, URDF)
Before this commit: robot jackal, 0 links, 0 joints
Links:
- added link $(arg mocap_frame_id)
Joints:
- added joint base_mocap_joint: type fixed, parent $(arg mocap_mount), child $(arg mocap_frame_id), origin xyz=$(arg mocap_xyz) rpy=$(arg mocap_rpy)
