Commit message: customization

File: jackal_description/urdf/jackal.urdf.xacro (robot description, xacro)
@@ -87,4 +87,10 @@
     <origin xyz="0 0 0" rpy="0 0 0" />
     <parent link="base_link"/>
+    <child link="base_footprint" />
+  </joint>
+  <link name="base_footprint"></link>
+  <joint name="footprint_joint" type="fixed">
+    <origin xyz="0 0 0" rpy="0 0 0" />
+    <parent link="base_footprint"/>
     <child link="chassis_link" />
   </joint>

Commit message: fixed simulation wheel slip

File: jackal_description/urdf/jackal.urdf.xacro (robot description, xacro)
@@ -17,4 +17,5 @@
   <xacro:property name="dummy_inertia" value="1e-09"/>
   <xacro:property name="mount_spacing" value="0.120" />
+  <xacro:arg name="wheel_slip" default="$(optenv JACKAL_WHEEL_SLIP 1)" />
   <material name="dark_grey"><color rgba="0.2 0.2 0.2 1.0" /></material>
   <material name="light_grey"><color rgba="0.4 0.4 0.4 1.0" /></material>
@@ -47,11 +48,15 @@
     <gazebo reference="${prefix}_wheel_link">
       <material>Gazebo/DarkGrey</material>
-      <selfCollide>false</selfCollide>
-      <mu1 value="0.5"/>
-      <mu2 value="0.5"/>
-      <!-- <kp value="10000000.0" />
-      <kd value="1" /> -->
-      <fdir1 value="1 0 0"/>
     </gazebo>
+    <xacro:unless value="$(arg wheel_slip)">
+      <gazebo reference="${prefix}_wheel_link">
+        <selfCollide>false</selfCollide>
+        <mu1 value="1.0"/>
+        <mu2 value="0.5"/>
+        <kp value="10000000.0" />
+        <kd value="1" />
+        <fdir1 value="1 0 0"/>
+      </gazebo>
+    </xacro:unless>
     <joint name="${prefix}_wheel_joint" type="continuous">
       <parent link="chassis_link"/>
@@ -106,10 +111,10 @@
     <inertial>
       <!-- Center of mass -->
-      <origin xyz="0.012  0.002 0.067" rpy="0 0 0"/>
+      <origin xyz="0.0 0.0 0.067" rpy="0 0 0"/>
       <mass value="16.523"/>
       <!-- Moments of inertia: ( chassis without wheels ) -->
       <inertia
-        ixx="0.3136" ixy="-0.0008" ixz="0.0164"
-        iyy="0.3922" iyz="-0.0009"
+        ixx="0.3136" ixy="0.0" ixz="0.0"
+        iyy="0.3922" iyz="0.0"
         izz="0.4485"/>
       </inertial>

Commit message: update collision box dimensions in URDF for improved accuracy

File: jackal_description/urdf/jackal.urdf.xacro (robot description, xacro)
@@ -135,5 +135,5 @@
         <origin xyz="0 0 ${chassis_height/2}"/>
         <geometry>
-          <box size="${chassis_length + 0.05} ${chassis_width + 0.10} ${chassis_height}"/>
+          <box size="${chassis_length + 0.07} ${chassis_width + 0.12} ${chassis_height}"/>
         </geometry>
       </collision>
