Commit message: correct env variable naming convention

File: jackal_description/urdf/accessories.urdf.xacro (robot description, xacro)
@@ -206,6 +206,6 @@
     <xacro:property name="name" value="$(optenv JACKAL_D435_NAME front)" />
     <xacro:property name="mount" value="$(optenv JACKAL_D435_MOUNT front)" />
-    <xacro:property name="camera_xyz" default="$(optenv JACKALD435_XYZ 0.042 0.0 0.0)" />
-    <xacro:property name="camera_rpy" default="$(optenv JACKALD435_RPY 0.0 0.0 0.0)" />
+    <xacro:property name="camera_xyz" default="$(optenv JACKAL_D435_XYZ 0.042 0.0 0.0)" />
+    <xacro:property name="camera_rpy" default="$(optenv JACKAL_D435_RPY 0.0 0.0 0.0)" />
     <xacro:property name="prefix" value="$(optenv JACKAL_D435_PREFIX ${mount})" />
     <xacro:property name="parent" value="$(optenv JACKAL_D435_PARENT ${mount}_mount)" />

Commit message: add people detector configuration to URDF with optional mounting properties

File: jackal_description/urdf/accessories.urdf.xacro (robot description, xacro)
@@ -200,4 +200,13 @@
   <xacro:include filename="$(find jackal_description)/urdf/accessories/camera_mount.urdf.xacro" />
   <!--xacro:include filename="$(find pointgrey_camera_description)/urdf/pointgrey_flea3.urdf.xacro" /-->
+  <xacro:if value="$(optenv JACKAL_PEOPLE_DETECTOR 0)">
+    <xacro:property name="mount" value="$(optenv JACKAL_PEOPLE_DETECTOR_MOUNT front)" />
+    <xacro:property name="prefix" value="$(optenv JACKAL_PEOPLE_DETECTOR_PREFIX ${mount})" />
+    <xacro:property name="parent" value="$(optenv JACKAL_PEOPLE_DETECTOR_PARENT ${mount}_mount)" />
+    <xacro:property name="tilt" value="$(optenv JACKAL_PEOPLE_DETECTOR_TILT 0)" />
+    <xacro:property name="xyz" value="$(optenv JACKAL_PEOPLE_DETECTOR_XYZ 0 0 0)" />
+    <xacro:property name="rpy" value="$(optenv JACKAL_PEOPLE_DETECTOR_RPY 0 0 0)" />
+    <xacro:include filename="$(find jackal_description)/urdf/accessories/people_detector.urdf.xacro" />
+  </xacro:if>
   <!-- If enabled, generate the d435 camera payload. -->
   <xacro:property name="d435" value="$(optenv JACKAL_D435 0)" />
