Commit message: add collision sensor configuration and lidar type selection to URDF

File: jackal_description/urdf/accessories/hokuyo_ust10.urdf.xacro (robot description, xacro)
@@ -14,5 +14,5 @@
       </link>
       <gazebo reference="${frame}">
-        <sensor type="ray" name="${frame}">
+        <sensor type="${lidar_type}" name="${frame}">
           <pose>0 0 0 0 0 0</pose>
           <visualize>false</visualize>

File: jackal_description/urdf/jackal.urdf.xacro (robot description, xacro)
@@ -5,4 +5,6 @@
   <xacro:arg name="prefix" default="" />
   <xacro:arg name="use_gazebo_controllers" default="True" />
+  <xacro:arg name="use_collision_sensor" default="False" />
+  <xacro:arg name="use_lidar_gpu" default="True" />
   <xacro:arg name="gazebo_controllers" default="$(find jackal_control)/config/control.yaml" />
   <xacro:property name="PI" value="3.1415926535897931" />
@@ -23,4 +25,6 @@
   <material name="yellow"><color rgba="0.8 0.8 0.0 1.0" /></material>
   <material name="black"><color rgba="0.15 0.15 0.15 1.0" /></material>
+  <xacro:property name="use_lidar_gpu" value="$(arg use_lidar_gpu)" />
+  <xacro:property name="lidar_type" value="${'gpu_ray' if use_lidar_gpu else 'ray'}" />
   <xacro:macro name="wheel" params="prefix *joint_pose">
     <link name="${prefix}_wheel_link">
@@ -121,4 +125,19 @@
       </inertial>
   </link>
+  <xacro:if value="$(arg use_collision_sensor)">
+    <joint name="collision_link_joint" type="fixed">
+      <origin xyz="0 0 0" rpy="0 0 0" />
+      <parent link="chassis_link"/>
+      <child link="collision_link" />
+    </joint>
+    <link name="collision_link">
+      <collision>
+        <origin xyz="0 0 ${chassis_height/2}"/>
+        <geometry>
+          <box size="${chassis_length + 0.05} ${chassis_width + 0.10} ${chassis_height}"/>
+        </geometry>
+      </collision>
+    </link>
+  </xacro:if>
   <xacro:unless value="$(optenv JACKAL_FRONT_ACCESSORY_FENDER 0)">
     <link name="front_fender_link">

Commit message: update lidar GPU usage flag and adjust sample size in URDF for consistency

File: jackal_description/urdf/accessories/hokuyo_ust10.urdf.xacro (robot description, xacro)
@@ -2,5 +2,5 @@
 <robot xmlns:xacro="http://ros.org/wiki/xacro">
   <xacro:macro name="hokuyo_ust10_mount" params="prefix topic parent_link *origin">
-    <xacro:macro name="hokuyo_ust10" params="frame:=laser topic:=scan sample_size:=720 update_rate:=30
+    <xacro:macro name="hokuyo_ust10" params="frame:=laser topic:=scan sample_size:=360 update_rate:=30
                min_angle:=-3.1416 max_angle:=3.1416 min_range:=0.1 max_range:=30.0 robot_namespace:=/">
       <link name="${frame}">

File: jackal_description/urdf/jackal.urdf.xacro (robot description, xacro)
@@ -6,5 +6,5 @@
   <xacro:arg name="use_gazebo_controllers" default="True" />
   <xacro:arg name="use_collision_sensor" default="False" />
-  <xacro:arg name="use_lidar_gpu" default="True" />
+  <xacro:arg name="use_lidar_gpu" default="False" />
   <xacro:arg name="gazebo_controllers" default="$(find jackal_control)/config/control.yaml" />
   <xacro:property name="PI" value="3.1415926535897931" />
